Commit message: Convert science system to position control

File: install/science_description/share/science_description/urdf/science_2026.urdf.xacro (robot description, xacro)
@@ -1,143 +1 @@
-<?xml version="1.0"?>
-<robot name="science_2026" xmlns:xacro="http://www.ros.org/wiki/xacro">
-  <link name="base_link">
-    <visual>
-      <origin xyz="0 0 0.025" rpy="0 0 0"/>
-      <geometry>
-        <box size="0.12 0.12 0.05"/>
-      </geometry>
-    </visual>
-  </link>
-  <link name="base_link_1">
-    <visual>
-      <origin xyz="0 0 0.05" rpy="0 0 0"/>
-      <geometry>
-        <cylinder radius="0.03" length="0.10"/>
-      </geometry>
-    </visual>
-  </link>
-  <link name="shoulder_link">
-    <visual>
-      <origin xyz="0.10 0 0" rpy="0 0 0"/>
-      <geometry>
-        <box size="0.20 0.04 0.04"/>
-      </geometry>
-    </visual>
-  </link>
-  <link name="elbow_link">
-    <visual>
-      <origin xyz="0.10 0 0" rpy="0 0 0"/>
-      <geometry>
-        <box size="0.20 0.03 0.03"/>
-      </geometry>
-    </visual>
-  </link>
-  <!-- Main wrist housing -->
-  <link name="wrist_roll_link">
-    <visual>
-      <origin xyz="0.025 0 0" rpy="0 0 0"/>
-      <geometry>
-        <box size="0.05 0.06 0.06"/>
-      </geometry>
-    </visual>
-    <visual>
-      <origin xyz="0.025 0 0" rpy="0 1.5708 0"/>
-      <geometry>
-        <cylinder radius="0.018" length="0.05"/>
-      </geometry>
-    </visual>
-  </link>
-  <!-- Front/output wrist piece -->
-  <link name="wrist_twist_link">
-    <visual>
-      <origin xyz="0.02 0 0" rpy="0 0 0"/>
-      <geometry>
-        <box size="0.04 0.045 0.045"/>
-      </geometry>
-    </visual>
-  </link>
-  <!-- Simple claw visual -->
-  <link name="claw_link">
-    <visual>
-      <origin xyz="0.03 0 0" rpy="0 0 0"/>
-      <geometry>
-        <box size="0.06 0.02 0.02"/>
-      </geometry>
-    </visual>
-  </link>
-  <joint name="base_yaw" type="revolute">
-    <parent link="base_link"/>
-    <child link="base_link_1"/>
-    <origin xyz="0 0 0.05" rpy="0 0 0"/>
-    <axis xyz="0 0 1"/>
-    <limit lower="-3.14" upper="3.14" effort="10" velocity="1.0"/>
-  </joint>
-  <!-- Zero position now starts 45 degrees upward -->
-  <joint name="shoulder_extension" type="revolute">
-    <parent link="base_link_1"/>
-    <child link="shoulder_link"/>
-    <origin xyz="0 0 0.10" rpy="0 -0.785398 0"/>
-    <axis xyz="0 1 0"/>
-    <limit lower="-1.57" upper="1.57" effort="10" velocity="0.2"/>
-  </joint>
-  <joint name="elbow_extension" type="revolute">
-    <parent link="shoulder_link"/>
-    <child link="elbow_link"/>
-    <origin xyz="0.20 0 0" rpy="0 0 0"/>
-    <axis xyz="0 1 0"/>
-    <limit lower="-1.57" upper="1.57" effort="10" velocity="0.2"/>
-  </joint>
-  <!-- Wrist module starts at forearm tip -->
-  <joint name="wrist_roll" type="revolute">
-    <parent link="elbow_link"/>
-    <child link="wrist_roll_link"/>
-    <origin xyz="0.20 0 0" rpy="0 0 0"/>
-    <axis xyz="0 1 0"/>
-    <limit lower="-1.57" upper="1.57" effort="10" velocity="0.5"/>
-  </joint>
-  <!-- Twist joint is almost co-located with wrist housing -->
-  <joint name="wrist_twist" type="revolute">
-    <parent link="wrist_roll_link"/>
-    <child link="wrist_twist_link"/>
-    <origin xyz="0.03 0 0" rpy="0 0 0"/>
-    <axis xyz="1 0 0"/>
-    <limit lower="-1.57" upper="1.57" effort="10" velocity="0.5"/>
-  </joint>
-  <!-- Claw attached after wrist twist -->
-  <joint name="claw" type="revolute">
-    <parent link="wrist_twist_link"/>
-    <child link="claw_link"/>
-    <origin xyz="0.04 0 0" rpy="0 0 0"/>
-    <axis xyz="0 1 0"/>
-    <limit lower="-1.57" upper="1.57" effort="10" velocity="0.5"/>
-  </joint>
-    <ros2_control name="Science2026Hardware" type="system">
-    <hardware>
-      <plugin>science_2026/Science2026System</plugin>
-    </hardware>
-    <joint name="base_yaw">
-      <command_interface name="velocity"/>
-      <state_interface name="position"/>
-    </joint>
-    <joint name="shoulder_extension">
-      <command_interface name="velocity"/>
-      <state_interface name="position"/>
-    </joint>
-    <joint name="elbow_extension">
-      <command_interface name="velocity"/>
-      <state_interface name="position"/>
-    </joint>
-    <joint name="wrist_roll">
-      <command_interface name="velocity"/>
-      <state_interface name="position"/>
-    </joint>
-    <joint name="wrist_twist">
-      <command_interface name="velocity"/>
-      <state_interface name="position"/>
-    </joint>
-    <joint name="claw">
-      <command_interface name="velocity"/>
-      <state_interface name="position"/>
-    </joint>
-  </ros2_control>
-</robot>
+/home/ibrahim/tasc_science/src/science_description/urdf/science_2026.urdf.xacro

File: src/science_description/urdf/science_2026.urdf.xacro (robot description, xacro)
@@ -117,25 +117,25 @@
     </hardware>
     <joint name="base_yaw">
-      <command_interface name="velocity"/>
+      <command_interface name="position"/>
       <state_interface name="position"/>
     </joint>
     <joint name="shoulder_extension">
-      <command_interface name="velocity"/>
+      <command_interface name="position"/>
       <state_interface name="position"/>
     </joint>
     <joint name="elbow_extension">
-      <command_interface name="velocity"/>
+      <command_interface name="position"/>
       <state_interface name="position"/>
     </joint>
     <joint name="wrist_roll">
-      <command_interface name="velocity"/>
+      <command_interface name="position"/>
       <state_interface name="position"/>
     </joint>
     <joint name="wrist_twist">
-      <command_interface name="velocity"/>
+      <command_interface name="position"/>
       <state_interface name="position"/>
     </joint>
     <joint name="claw">
-      <command_interface name="velocity"/>
+      <command_interface name="position"/>
       <state_interface name="position"/>
     </joint>
