Commit message: Full science repo overhaul. New URDF + new hardware interface + polished controls

File: src/science_description/urdf/science_2026.urdf.xacro (robot description, xacro)
@@ -1,140 +1,280 @@
 <?xml version="1.0"?>
-<robot name="science_2026" xmlns:xacro="http://www.ros.org/wiki/xacro">
+<robot name="science_system" xmlns:xacro="http://www.ros.org/wiki/xacro">
+  <!-- ========================================================= -->
+  <!-- MATERIALS                                                 -->
+  <!-- ========================================================= -->
+  <material name="dark_gray">
+    <color rgba="0.25 0.25 0.25 1.0"/>
+  </material>
+  <material name="light_gray">
+    <color rgba="0.70 0.70 0.70 1.0"/>
+  </material>
+  <material name="black">
+    <color rgba="0.10 0.10 0.10 1.0"/>
+  </material>
+  <material name="blue">
+    <color rgba="0.15 0.35 0.75 1.0"/>
+  </material>
+  <material name="green">
+    <color rgba="0.15 0.55 0.30 1.0"/>
+  </material>
+  <material name="red">
+    <color rgba="0.90 0.10 0.10 1.0"/>
+  </material>
+  <material name="yellow">
+    <color rgba="1.0 0.80 0.05 1.0"/>
+  </material>
+  <material name="beaker_glass">
+    <color rgba="0.80 0.90 1.0 0.75"/>
+  </material>
+  <!-- ========================================================= -->
+  <!-- FIXED BASE                                                -->
+  <!-- ========================================================= -->
+  <!--
+    Fixed frame for the science mechanism.
+    The linear actuator housing is above the auger.
+    The beaker tray is also supported from this fixed structure,
+    so the tray does not move when the auger moves vertically.
+  -->
   <link name="base_link">
-    <visual>
-      <origin xyz="0 0 0.025" rpy="0 0 0"/>
-      <geometry>
-        <box size="0.12 0.12 0.05"/>
-      </geometry>
-    </visual>
-  </link>
-  <link name="base_link_1">
-    <visual>
-      <origin xyz="0 0 0.05" rpy="0 0 0"/>
-      <geometry>
-        <cylinder radius="0.03" length="0.10"/>
-      </geometry>
-    </visual>
-  </link>
-  <link name="shoulder_link">
-    <visual>
-      <origin xyz="0.10 0 0" rpy="0 0 0"/>
-      <geometry>
-        <box size="0.20 0.04 0.04"/>
-      </geometry>
-    </visual>
-  </link>
-  <link name="elbow_link">
-    <visual>
-      <origin xyz="0.10 0 0" rpy="0 0 0"/>
-      <geometry>
-        <box size="0.20 0.03 0.03"/>
-      </geometry>
-    </visual>
-  </link>
-  <!-- Main wrist housing -->
-  <link name="wrist_roll_link">
-    <visual>
-      <origin xyz="0.025 0 0" rpy="0 0 0"/>
-      <geometry>
-        <box size="0.05 0.06 0.06"/>
-      </geometry>
-    </visual>
-    <visual>
-      <origin xyz="0.025 0 0" rpy="0 1.5708 0"/>
-      <geometry>
-        <cylinder radius="0.018" length="0.05"/>
-      </geometry>
-    </visual>
-  </link>
-  <!-- Front/output wrist piece -->
-  <link name="wrist_twist_link">
-    <visual>
-      <origin xyz="0.02 0 0" rpy="0 0 0"/>
-      <geometry>
-        <box size="0.04 0.045 0.045"/>
-      </geometry>
-    </visual>
-  </link>
-  <!-- Simple claw visual -->
-  <link name="claw_link">
-    <visual>
-      <origin xyz="0.03 0 0" rpy="0 0 0"/>
-      <geometry>
-        <box size="0.06 0.02 0.02"/>
-      </geometry>
-    </visual>
-  </link>
-  <joint name="base_yaw" type="revolute">
+    <!-- Upper mounting plate -->
+    <visual>
+      <origin xyz="0 0 0" rpy="0 0 0"/>
+      <geometry>
+        <box size="0.50 0.30 0.05"/>
+      </geometry>
+      <material name="dark_gray"/>
+    </visual>
+    <!-- Fixed linear actuator housing -->
+    <visual>
+      <origin xyz="-0.16 0 -0.125" rpy="0 0 0"/>
+      <geometry>
+        <cylinder radius="0.04" length="0.20"/>
+      </geometry>
+      <material name="black"/>
+    </visual>
+    <!-- Fixed vertical support for the beaker tray -->
+    <visual>
+      <origin xyz="0.16 0 -0.33" rpy="0 0 0"/>
+      <geometry>
+        <box size="0.05 0.05 0.60"/>
+      </geometry>
+      <material name="dark_gray"/>
+    </visual>
+    <!-- Fixed servo housing near the tray -->
+    <visual>
+      <origin xyz="0.16 0 -0.61" rpy="0 0 0"/>
+      <geometry>
+        <box size="0.10 0.08 0.08"/>
+      </geometry>
+      <material name="black"/>
+    </visual>
+  </link>
+  <!-- ========================================================= -->
+  <!-- MOVING AUGER CARRIAGE                                     -->
+  <!-- ========================================================= -->
+  <!--
+    This link moves vertically with the linear actuator.
+    Only the auger assembly is attached to this link.
+    The beaker tray is not attached to this link.
+  -->
+  <link name="auger_carriage_link">
+    <!-- Moving actuator rod -->
+    <visual>
+      <origin xyz="0 0 0.10" rpy="0 0 0"/>
+      <geometry>
+        <cylinder radius="0.02" length="0.25"/>
+      </geometry>
+      <material name="light_gray"/>
+    </visual>
+    <!-- Auger motor housing -->
+    <visual>
+      <origin xyz="0 0 -0.08" rpy="0 0 0"/>
+      <geometry>
+        <cylinder radius="0.06" length="0.12"/>
+      </geometry>
+      <material name="blue"/>
+    </visual>
+    <!-- Motor mounting plate -->
+    <visual>
+      <origin xyz="0 0 -0.015" rpy="0 0 0"/>
+      <geometry>
+        <box size="0.14 0.14 0.03"/>
+      </geometry>
+      <material name="dark_gray"/>
+    </visual>
+  </link>
+  <!-- ========================================================= -->
+  <!-- ROTATING AUGER                                            -->
+  <!-- ========================================================= -->
+  <link name="auger_link">
+    <!-- Main auger shaft -->
+    <visual>
+      <origin xyz="0 0 -0.24" rpy="0 0 0"/>
+      <geometry>
+        <cylinder radius="0.018" length="0.48"/>
+      </geometry>
+      <material name="light_gray"/>
+    </visual>
+    <!--
+      Asymmetric red marker.
+      A plain cylinder looks unchanged while rotating.
+      This marker makes auger rotation visible in RViz.
+    -->
+    <visual>
+      <origin xyz="0.055 0 -0.07" rpy="0 0 0"/>
+      <geometry>
+        <box size="0.11 0.025 0.025"/>
+      </geometry>
+      <material name="red"/>
+    </visual>
+    <!-- Upper auger blade -->
+    <visual>
+      <origin xyz="0.035 0 -0.16" rpy="0.25 0 0.55"/>
+      <geometry>
+        <box size="0.10 0.025 0.018"/>
+      </geometry>
+      <material name="light_gray"/>
+    </visual>
+    <!-- Middle auger blade -->
+    <visual>
+      <origin xyz="-0.025 0.025 -0.27" rpy="-0.25 0 2.10"/>
+      <geometry>
+        <box size="0.10 0.025 0.018"/>
+      </geometry>
+      <material name="light_gray"/>
+    </visual>
+    <!-- Lower auger blade -->
+    <visual>
+      <origin xyz="0 -0.035 -0.38" rpy="0.25 0 -1.05"/>
+      <geometry>
+        <box size="0.10 0.025 0.018"/>
+      </geometry>
+      <material name="light_gray"/>
+    </visual>
+    <!-- Drill tip -->
+    <visual>
+      <origin xyz="0 0 -0.50" rpy="0 0 0"/>
+      <geometry>
+        <cylinder radius="0.045" length="0.04"/>
+      </geometry>
+      <material name="dark_gray"/>
+    </visual>
+  </link>
+  <!-- ========================================================= -->
+  <!-- FIXED-HEIGHT ROTATING BEAKER TRAY                          -->
+  <!-- ========================================================= -->
+  <!--
+    The tray rotates but does not move vertically.
+    Its joint is connected directly to base_link rather than
+    auger_carriage_link.
+  -->
+  <link name="beaker_tray_link">
+    <!-- Circular tray -->
+    <visual>
+      <origin xyz="0 0 -0.025" rpy="0 0 0"/>
+      <geometry>
+        <cylinder radius="0.15" length="0.05"/>
+      </geometry>
+      <material name="green"/>
+    </visual>
+    <!-- Tray direction marker -->
+    <visual>
+      <origin xyz="0.10 0 0.01" rpy="0 0 0"/>
+      <geometry>
+        <box size="0.10 0.018 0.018"/>
+      </geometry>
+      <material name="yellow"/>
+    </visual>
+    <!-- Beaker at 0 degrees -->
+    <visual>
+      <origin xyz="0.10 0 0.065" rpy="0 0 0"/>
+      <geometry>
+        <cylinder radius="0.025" length="0.11"/>
+      </geometry>
+      <material name="beaker_glass"/>
+    </visual>
+    <!-- Beaker at 90 degrees -->
+    <visual>
+      <origin xyz="0 0.10 0.065" rpy="0 0 0"/>
+      <geometry>
+        <cylinder radius="0.025" length="0.11"/>
+      </geometry>
+      <material name="beaker_glass"/>
+    </visual>
+    <!-- Beaker at 180 degrees -->
+    <visual>
+      <origin xyz="-0.10 0 0.065" rpy="0 0 0"/>
+      <geometry>
+        <cylinder radius="0.025" length="0.11"/>
+      </geometry>
+      <material name="beaker_glass"/>
+    </visual>
+  </link>
+  <!-- ========================================================= -->
+  <!-- JOINTS                                                    -->
+  <!-- ========================================================= -->
+  <!--
+    Linear actuator moving only the auger carriage.
+    Positive joint motion is currently along +Z.
+    Change the axis to 0 0 -1 if positive commands should move
+    the auger downward.
+    URDF requires limits for a prismatic joint.
+    These broad limits are primarily for URDF validity.
+  -->
+  <joint name="science_lift_joint" type="prismatic">
     <parent link="base_link"/>
-    <child link="base_link_1"/>
-    <origin xyz="0 0 0.05" rpy="0 0 0"/>
+    <child link="auger_carriage_link"/>
+    <origin xyz="-0.16 0 -0.25" rpy="0 0 0"/>
     <axis xyz="0 0 1"/>
-    <limit lower="-3.14" upper="3.14" effort="10" velocity="1.0"/>
+    <limit
+      lower="-1.0"
+      upper="1.0"
+      effort="1000.0"
+      velocity="1.0"/>
   </joint>
-  <!-- Zero position now starts 45 degrees upward -->
-  <joint name="shoulder_extension" type="revolute">
-    <parent link="base_link_1"/>
-    <child link="shoulder_link"/>
-    <origin xyz="0 0 0.10" rpy="0 -0.785398 0"/>
-    <axis xyz="0 1 0"/>
-    <limit lower="-1.57" upper="1.57" effort="10" velocity="0.2"/>
+  <!--
+    Continuous Phidget stepper rotation.
+    The red marker and uneven blades make rotation visible in RViz.
+  -->
+  <joint name="auger_spin_joint" type="continuous">
+    <parent link="auger_carriage_link"/>
+    <child link="auger_link"/>
+    <origin xyz="0 0 -0.14" rpy="0 0 0"/>
+    <axis xyz="0 0 1"/>
   </joint>
-  <joint name="elbow_extension" type="revolute">
-    <parent link="shoulder_link"/>
-    <child link="elbow_link"/>
-    <origin xyz="0.20 0 0" rpy="0 0 0"/>
-    <axis xyz="0 1 0"/>
-    <limit lower="-1.57" upper="1.57" effort="10" velocity="0.2"/>
+  <!--
+    Beaker tray remains at a fixed height and only rotates.
+    Intended servo positions:
+      0 degrees   = 0.0 radians
+      90 degrees  = 1.5708 radians
+      180 degrees = 3.14159 radians
+  -->
+  <joint name="beaker_tray_joint" type="continuous">
+    <parent link="base_link"/>
+    <child link="beaker_tray_link"/>
+    <!-- Positioned near the bottom level of the lowered auger -->
+    <origin xyz="0.16 0 -0.65" rpy="0 0 0"/>
+    <axis xyz="0 0 1"/>
   </joint>
-  <!-- Wrist module starts at forearm tip -->
-  <joint name="wrist_roll" type="revolute">
-    <parent link="elbow_link"/>
-    <child link="wrist_roll_link"/>
-    <origin xyz="0.20 0 0" rpy="0 0 0"/>
-    <axis xyz="0 1 0"/>
-    <limit lower="-1.57" upper="1.57" effort="10" velocity="0.5"/>
-  </joint>
-  <!-- Twist joint is almost co-located with wrist housing -->
-  <joint name="wrist_twist" type="revolute">
-    <parent link="wrist_roll_link"/>
-    <child link="wrist_twist_link"/>
-    <origin xyz="0.03 0 0" rpy="0 0 0"/>
-    <axis xyz="1 0 0"/>
-    <limit lower="-1.57" upper="1.57" effort="10" velocity="0.5"/>
-  </joint>
-  <!-- Claw attached after wrist twist -->
-  <joint name="claw" type="revolute">
-    <parent link="wrist_twist_link"/>
-    <child link="claw_link"/>
-    <origin xyz="0.04 0 0" rpy="0 0 0"/>
-    <axis xyz="0 1 0"/>
-    <limit lower="-1.57" upper="1.57" effort="10" velocity="0.5"/>
-  </joint>
-    <ros2_control name="Science2026Hardware" type="system">
+  <!-- ========================================================= -->
+  <!-- ROS 2 CONTROL                                             -->
+  <!-- ========================================================= -->
+  <ros2_control name="ScienceHardware" type="system">
     <hardware>
       <plugin>science_2026/Science2026System</plugin>
     </hardware>
-    <joint name="base_yaw">
-      <command_interface name="position"/>
+    <!-- Linear actuator up and down -->
+    <joint name="science_lift_joint">
+      <command_interface name="velocity"/>
       <state_interface name="position"/>
     </joint>
-    <joint name="shoulder_extension">
-      <command_interface name="position"/>
+    <!-- Continuous auger rotation -->
+    <joint name="auger_spin_joint">
+      <command_interface name="velocity"/>
       <state_interface name="position"/>
     </joint>
-    <joint name="elbow_extension">
-      <command_interface name="position"/>
-      <state_interface name="position"/>
-    </joint>
-    <joint name="wrist_roll">
-      <command_interface name="position"/>
-      <state_interface name="position"/>
-    </joint>
-    <joint name="wrist_twist">
-      <command_interface name="position"/>
-      <state_interface name="position"/>
-    </joint>
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